Commit message: fix(tcp): 统一以 URDF 定义 TCP，移除冗余配置 - 更新 `piper_description.urdf` 添加 `link_tcp` 定义 - config.yaml 移除 `tcp_offset` 配置 - piper_interface 相关代码调整以适配 URDF 定义的 TCP docs: 更新 README 中的 EEF/TCP 配置说明

File: piper_ros/src/piper_description/urdf/piper_description.urdf (robot description, URDF)
Before this commit: robot piper_description, 8 links, 7 joints
Links:
- added link link_tcp
Joints:
- added joint joint_tcp: type fixed, parent link6, child link_tcp, origin xyz=0 0.018 0.13181 rpy=0 0 0

File: piper_ros/src/piper_moveit/piper_with_gripper_moveit/config/gazebo_piper_description.urdf (robot description, URDF)
Before this commit: robot piper_description, 9 links, 8 joints
Links:
- removed link link7
- removed link link8
- added link link_tcp
- added link world
- link base_link: mass 0.16229 -> 0.162290652295194; geometry collision mesh filename=package://piper_description/processed_meshes/visual/base_li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; visual mesh filename=package://piper_description/meshes/base_link.STL
- link link1: geometry collision mesh filename=package://piper_description/processed_meshes/visual/link1.S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; visual mesh filename=package://piper_description/meshes/link1.STL
- link link2: geometry collision mesh filename=package://piper_description/processed_meshes/visual/link2.S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; visual mesh filename=package://piper_description/meshes/link2.STL
- link link3: mass 0.259293339150458 -> 0.259293309425469; geometry collision mesh filename=package://piper_description/processed_meshes/visual/link3.S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; visual mesh filename=package://piper_description/meshes/link3.STL
- link link4: geometry collision mesh filename=package://piper_description/processed_meshes/visual/link4.S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; visual mesh filename=package://piper_description/meshes/link4.STL
- link link5: mass 0.136390779564153 -> 0.136390779513211; geometry collision mesh filename=package://piper_description/processed_meshes/visual/link5.S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; visual mesh filename=package://piper_description/meshes/link5.STL
- link link6: mass 0.223574803988609 -> 0.297734657028244; geometry collision mesh filename=package://piper_description/processed_meshes/visual/link6.S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; visual mesh filename=package://piper_description/meshes/link6.STL
Joints:
- removed joint joint7
- removed joint joint8
- added joint joint_tcp: type fixed, parent link6, child link_tcp, origin xyz=0 0.018 0.13181 rpy=0 0 0
- added joint world_joint: type fixed, parent world, child base_link

Commit message: fix(urdf): 关节三和关节五反向问题 fix(controller): 末端执行器命令后增加延时 fix(task_manager): 任务完成后夹爪复位 fix(piper_start): 注释掉旧版本机械臂回零代码

File: piper_ros/src/piper_description/urdf/piper_description.urdf (robot description, URDF)
Before this commit: robot piper_description, 9 links, 8 joints
Joints:
- joint joint3: axis 0 0 1 -> 0 0 -1; limit lower=0 upper=2.967 effort=100 velocity=5 -> lower=-2.967 upper=0 effort=100 velocity=5
- joint joint5: axis 0 0 1 -> 0 0 -1
